File: PCB/_autosave-Power.kicad_sch (KiCad schematic)
At the start: 27 parts, among them U2 XL4005E1, U3 NCP1117-3.3_SOT223

Commit message: Minor Schematic tweaks like - Adding pull up resistors to the spare GPIO pins - Renaming some Global Labels - Labeling all the pins on the STM32 correctly
Parts:
- renumbered H6 to H5, H5 to H6
Changed lines of the file:
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@@
 		(dnp no)
 		(fields_autoplaced yes)
-		(property "Reference" "H6"
+		(property "Reference" "H5"
 			(at 54.61 170.1799 90)
 			(show_name no)
@@
 			(project "Arm_Controller"
 				(path "/2323d903-32ae-4da3-a89f-487023e10892/2ee041d2-835d-4fc4-b3fc-43e28808df04"
-					(reference "H6")
+					(reference "H5")
 					(unit 1)
 				)
@@
 		(dnp no)
 		(fields_autoplaced yes)
-		(property "Reference" "H5"
+		(property "Reference" "H6"
 			(at 54.61 165.0999 90)
 			(show_name no)
@@
 			(project "Arm_Controller"
 				(path "/2323d903-32ae-4da3-a89f-487023e10892/2ee041d2-835d-4fc4-b3fc-43e28808df04"
-					(reference "H5")
-					(unit 1)
-				)
+					(reference "H6")
+					(unit 1)
+				)
